File: servo/pcb/main.kicad_sch (KiCad schematic)
At the start: 14 parts, among them J1 Conn_01x03_Socket, J2 Conn_01x03_Socket, J3 Conn_01x03_Socket, SW1 SW_Omron_B3FS, SW2 SW_Omron_B3FS, SW3 SW_Omron_B3FS, U1 Pico

Commit message: P配線した
Parts:
- added J4, J5: Conn_01x02_Socket, Connector_PinSocket_2.54mm:PinSocket_1x02_P2.54mm_Vertical, symbol Connector:Conn_01x02_Socket
- added Q1: FQP27P06, Package_TO_SOT_THT:TO-92_Inline_Wide, symbol Transistor_FET:FQP27P06
- SW1, SW2, SW3: footprint Button_Switch_SMD:SW_SPST_Omron_B3FS-100xP -> Button_Switch_THT:SW_PUSH_6mm
Connections:
- net GND: now also J5.1 (Pin_1)
- net VCC: now also U1.39 (VSYS), J5.2 (Pin_2), Q1.3 (S); no longer U1.40 (VBUS)
- new net: J4.1 (Pin_1), Q1.1 (G), U1.40 (VBUS)
- new net: J4.2 (Pin_2), Q1.2 (D)
- no-connect marks 32 -> 31
Other:
- moved on the sheet: C1, C2
