File: servo/pcb/main.kicad_pcb (KiCad board)
At the start: 2 copper layers, 11 parts, among them J1 Conn_01x03_Socket, J2 Conn_01x03_Socket, J3 Conn_01x03_Socket, SW1 SW_Omron_B3FS, SW2 SW_Omron_B3FS, SW3 SW_Omron_B3FS, U1 Pico

Commit message: P配線した
Parts:
- added H2: MountingHole, MountingHole:MountingHole_3.2mm_M3, F.Cu at (53.8, 113.5)
- added H3: MountingHole, MountingHole:MountingHole_3.2mm_M3, F.Cu at (53.8, 53.8)
- added H4: MountingHole, MountingHole:MountingHole_3.2mm_M3, F.Cu at (103.3, 53.8)
- added J4: Conn_01x02_Socket, Connector_PinSocket_2.54mm:PinSocket_1x02_P2.54mm_Vertical, F.Cu at (102.1, 62.7)
- added J5: Conn_01x02_Socket, Connector_PinSocket_2.54mm:PinSocket_1x02_P2.54mm_Vertical, F.Cu at (102.1, 71.6)
- added Q1: FQP27P06, Package_TO_SOT_THT:TO-92_Inline_Wide, F.Cu at (95.7, 55.1)
- SW1, SW2, SW3: footprint Button_Switch_SMD:SW_SPST_Omron_B3FS-100xP -> Button_Switch_THT:SW_PUSH_6mm
- moved TP1 37.4 mm to (85.6, 113.5)
- moved J2 33.4 mm to (93.2, 108.4)
- moved SW3 22.3 mm to (54.8, 94.8)
- moved SW2 17.3 mm to (54.8, 76.8)
- moved J3 16.5 mm to (64.0, 108.4)
- moved SW1 15.2 mm to (54.8, 60.8)
- moved C2 10.4 mm to (94.5, 65.2)
- moved H1 9.31 mm to (103.3, 113.5)
- moved U1 8.79 mm to (77.9, 76.7)
- moved C1 8.11 mm to (94.5, 72.9)
- moved J1 5.91 mm to (97.0, 83.0)
Connections:
- U1 pad 39: unconnected-(U1-VSYS-Pad39) -> VCC
- U1 pad 40: VCC -> Net-(J4-Pin_1)
Routing:
- net Net-(J2-Pin_3): track 0.00 -> 50.0 mm
- net Net-(U1-GPIO4): track 0.00 -> 45.1 mm
- net Net-(J3-Pin_3): track 0.00 -> 40.9 mm
- net Net-(U1-GPIO3): track 0.00 -> 30.6 mm
- net Net-(J1-Pin_2): track 0.00 -> 29.6 mm
- net Net-(J4-Pin_1): track 0.00 -> 20.9 mm
- net Net-(J1-Pin_3): track 0.00 -> 20.6 mm
- net Net-(U1-GPIO2): track 0.00 -> 17.1 mm
- net Net-(J4-Pin_2): track 0.00 -> 11.2 mm
- net VCC: track 0.00 -> 11.0 mm
- added copper zone on B.Cu, net GND
- added copper zone on F.Cu, net VCC
Other:
- board outline added: 57.2 x 68.6 mm
- board text added: "3V3"
- board text added: "GND"
- board text added: "PWM"
- board text added: "Potention"
- board text added: "VCC"

Commit message: rev1
Parts:
- moved H1 3.65 mm to (106.0, 116.0)
- moved H4 2.66 mm to (106.0, 53.8)
- moved H2 2.51 mm to (54.0, 116.0)
Other:
- board size 57.2 x 68.6 mm -> 60 x 70 mm
Changed lines of the file:
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@@
     (grid_origin 50 50)
     (pcbplotparams
-      (layerselection 0x00010fc_ffffffff)
+      (layerselection 0x00010f0_ffffffff)
       (plot_on_all_layers_selection 0x0000000_00000000)
       (disableapertmacros false)
@@
       (plotinvisibletext false)
       (sketchpadsonfab false)
-      (subtractmaskfromsilk false)
+      (subtractmaskfromsilk true)
       (outputformat 1)
       (mirror false)
-      (drillshape 1)
+      (drillshape 0)
       (scaleselection 1)
       (outputdirectory "")
@@
   (net 42 "Net-(J4-Pin_2)")
   (footprint "MountingHole:MountingHole_3.2mm_M3" (layer "F.Cu")
-    (at 103.34 113.5)
+    (at 106 116)
     (descr "Mounting Hole 3.2mm, no annular, M3")
     (tags "mounting hole 3.2mm no annular m3")
@@
   )
   (footprint "MountingHole:MountingHole_3.2mm_M3" (layer "F.Cu")
-    (at 103.34 53.81)
+    (at 106 53.81)
     (descr "Mounting Hole 3.2mm, no annular, M3")
     (tags "mounting hole 3.2mm no annular m3")
@@
   )
   (footprint "MountingHole:MountingHole_3.2mm_M3" (layer "F.Cu")
-    (at 53.81 113.5)
+    (at 54 116)
     (descr "Mounting Hole 3.2mm, no annular, M3")
     (tags "mounting hole 3.2mm no annular m3")
@@
       (net 5 "Net-(J2-Pin_3)") (pinfunction "1") (pintype "passive"))
   )
-  (gr_rect (start 50 50) (end 107.15 118.58)
+  (gr_rect (start 50 50) (end 110 120)
     (stroke (width 0.2) (type default)) (fill none) (layer "Edge.Cuts"))
   (gr_text "VCC" (at 58.89 112.23) (layer "F.SilkS")
@@
   )
   (dimension (type aligned) (layer "Dwgs.User")
-    (pts (xy 107.15 50) (xy 107.15 118.58))
+    (pts (xy 110 50) (xy 110 120))
     (height -11.43)
-    (gr_text "68.5800 mm" (at 116.88 84.29 90) (layer "Dwgs.User")
+    (gr_text "70.0000 mm" (at 119.73 85 90) (layer "Dwgs.User")
       (effects (font (size 1.5 1.5) (thickness 0.2)))
     )
@@
   )
   (dimension (type aligned) (layer "Dwgs.User")
-    (pts (xy 50 50) (xy 107.15 50))
+    (pts (xy 50 50) (xy 110 50))
     (height -8.89)
-    (gr_text "57.1500 mm" (at 78.575 39.41) (layer "Dwgs.User")
+    (gr_text "60.0000 mm" (at 80 39.41) (layer "Dwgs.User")
       (effects (font (size 1.5 1.5) (thickness 0.2)))
     )
@@
       (pts
         (xy 51 51)
-        (xy 106 51)
-        (xy 106 118)
-        (xy 51 118)
+        (xy 109 51)
+        (xy 109 119)
+        (xy 51 119)
       )
     )
@@
       (pts
         (xy 51 51)
-        (xy 106 51)
-        (xy 106 118)
-        (xy 51 118)
+        (xy 109 51)
+        (xy 109 119)
+        (xy 51 119)
       )
     )
